Commit message: update joint limit

File: aubo_ros2_description/urdf/aubo_i5.urdf.xacro (robot description, xacro)
@@ -56,5 +56,5 @@
     <child link="shoulder_Link" />
     <axis xyz="0 0 1" />
-    <limit lower="-3.04" upper="3.04" effort="0" velocity="0" />
+    <limit lower="-6.28" upper="6.28" effort="0" velocity="0" />
   </joint>
   <link name="upperArm_Link">
@@ -85,5 +85,5 @@
     <child link="upperArm_Link" />
     <axis xyz="0 0 1" />
-    <limit lower="-3.04" upper="3.04" effort="0" velocity="0" />
+    <limit lower="-6.28" upper="6.28" effort="0" velocity="0" />
   </joint>
   <link name="foreArm_Link">
@@ -114,5 +114,5 @@
     <child link="foreArm_Link" />
     <axis xyz="0 0 1" />
-    <limit lower="-3.04" upper="3.04" effort="0" velocity="0" />
+    <limit lower="-6.28" upper="6.28" effort="0" velocity="0" />
   </joint>
   <link name="wrist1_Link">
@@ -143,5 +143,5 @@
     <child link="wrist1_Link" />
     <axis xyz="0 0 1" />
-    <limit lower="-3.04" upper="3.04" effort="0" velocity="0" />
+    <limit lower="-6.28" upper="6.28" effort="0" velocity="0" />
   </joint>
   <link name="wrist2_Link">
@@ -172,5 +172,5 @@
     <child link="wrist2_Link" />
     <axis xyz="0 0 1" />
-    <limit lower="-3.04" upper="3.04" effort="0" velocity="0" />
+    <limit lower="-6.28" upper="6.28" effort="0" velocity="0" />
   </joint>
   <link name="wrist3_Link">
@@ -201,5 +201,5 @@
     <child link="wrist3_Link" />
     <axis xyz="0 0 1" />
-    <limit lower="-3.04" upper="3.04" effort="0" velocity="0" />
+    <limit lower="-6.28" upper="6.28" effort="0" velocity="0" />
   </joint>
   <link name="world" />
